File: hardware/main.brd (EAGLE design)
At the start: 160 x 100 mm, 38 parts, among them IC1 FT232RL, J1 POWER_JACKPTH_BREAD, M1 SERVO, M2 SERVO, M3 SERVO, P1 61729-1011BLF, X1 STEREOJACK

Commit message: Updated hardware files for eagle
Parts:
- removed C5: 10µF, rcl:C075-032X103
- removed C7: 0.1µF, rcl:C075-032X103
- removed IC1: FT232RL, ftdichip:SSOP28
- removed OK2: ILQ1, optocoupler:DIL16
- removed P1: 61729-1011BLF, Common-Parts-Library-Eagle:FCI_61729-1011BLF
- removed R3, R5, R7: 220Ω, rcl:0207/10
- removed U$12, U$13: PIRANHA_LED, Mel_Custom:LED_PIRANHA_5MM
- moved R1 73.7 mm to (39.4, 95.2), turned to 180 degrees
- moved M3 71.5 mm to (25.4, 77.5), turned to 90 degrees
- moved L1 70.8 mm to (26.7, 92.7), turned to 90 degrees
- moved C2 70.7 mm to (34.3, 95.2)
- moved U$1 70.7 mm to (44.5, 95.2), turned to 270 degrees
- moved M2 69.5 mm to (21.6, 77.5), turned to 90 degrees
- moved M1 67.8 mm to (17.8, 77.5), turned to 90 degrees
- moved C1 64.7 mm to (30.5, 95.2)
- moved U$9 63.7 mm to (64.8, 67.3), turned to 90 degrees
- moved J1 63.6 mm to (0.00, 96.5), turned to 270 degrees
- moved C3 61.6 mm to (8.89, 82.5)
- moved U$5 61.0 mm to (20.4, 86.6), turned to 0 degrees
- moved R2 60.5 mm to (20.3, 92.7)
- moved PAD2 59.8 mm to (22.9, 97.8)
- moved PAD1 58.5 mm to (17.8, 97.8)
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Connections:
- removed net N$20: OK2.16, U$2.RX1-1
- removed net N$28: C5.1, C7.1, IC1.20, OK2.10, OK2.14, P1.1
- removed net N$36: S1.2, U$2.A6
- removed net N$37: IC1.2, OK2.5, OK2.9
- removed net N$39: IC1.15, P1.3
- removed net N$40: IC1.16, P1.2
- removed net N$41: OK2.4, U$2.TX0-1
- removed net N$43: IC1.5, OK2.13
- removed net N$44: OK2.11, OK2.8, U$2.DTR
- removed net N$45: R5.1, U$13.+@0, U$13.+@1
- removed net N$46: R7.1, U$12.+@0, U$12.+@1
- removed net N$47: IC1.23, U$12.-@0, U$12.-@1
- removed net N$48: IC1.1, OK2.1
- removed net N$50: C5.2, C7.2, IC1.11, IC1.18, IC1.21, IC1.25, IC1.26, IC1.7, OK2.2, OK2.6, P1.4, R5.2, R7.2
- removed net N$52: IC1.22, U$13.-@0, U$13.-@1
- removed net VCCIO: IC1.4
- net N$15: now also S1.2, U$2.A1; no longer R3.1, U$6.LED2, U$7.LED2, U$8.LED2
- net N$19: no longer OK2.12
- net N$23: no longer S1.3
- net N$38: no longer OK2.3, OK2.7, R3.2, U$2.GND2, U$2.GND3, U$2.GND4
- net N$42: now also S1.3; no longer OK2.15, U$2.VCC1
Routing:
- net N$38: track 373.4 -> 206.3 mm
- net N$50: track 129.7 -> 0.00 mm
- net N$28: track 82.0 -> 0.00 mm
- net N$19: track 80.5 -> 0.00 mm
- net N$42: track 170.1 -> 108.3 mm, vias 1 -> 0
- net N$21: track 99.0 -> 41.4 mm
- net N$18: track 93.5 -> 41.2 mm, vias 1 -> 0
- net N$25: track 88.5 -> 42.7 mm
- net N$24: track 81.4 -> 37.9 mm
- net N$22: track 80.4 -> 44.4 mm
- net N$37: track 31.0 -> 0.00 mm
- net N$23: track 38.2 -> 7.62 mm
- net N$36: track 26.8 -> 0.00 mm
- net N$39: track 26.7 -> 0.00 mm
- net N$40: track 23.1 -> 0.00 mm
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Other:
- board size 160 x 100 mm -> 64.8 x 53 mm

Commit message: Updated hardware
Parts:
- added J2, J3: (no value), SparkFun-Connectors:1X01
- moved OK1 84.1 mm to (-14.0, -11.4)
- moved C1 79.5 mm to (-5.08, 24.1)
- moved C2 79.5 mm to (-1.27, 24.1)
- moved C3 79.5 mm to (-26.7, 11.4)
- moved C4 79.5 mm to (-30.5, 11.4)
- moved J1 79.5 mm to (-35.6, 25.4)
- moved L2 79.5 mm to (-24.8, 18.5)
- moved M1 79.5 mm to (-17.8, 6.35)
- moved M2 79.5 mm to (-14.0, 6.35)
- moved M3 79.5 mm to (-10.2, 6.35)
- moved PAD1 79.5 mm to (-17.8, 26.7)
- moved PAD2 79.5 mm to (-12.7, 26.7)
- moved R1 79.5 mm to (3.81, 24.1)
- moved R4 79.5 mm to (-21.6, 10.8)
- moved S1 79.5 mm to (19.1, -19.1)
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Connections:
- removed net N$19 (its old number): U$1.4
- removed net N$23: M1.2, M2.2, M3.2
- removed net N$38: C1.2, C2.2, C3.2, C4.2, J1.GND, J1.GNDBREAK, M1.3, M2.3, M3.3, OK1.3, PAD2.1, R1.3, R2.3, S1.1, U$1.3, U$2.GND, U$2.GND1, U$5.3, U$6.SW2, U$7.SW2, U$8.SW2, U$9.1, U$9.10, U$9.11, U$9.12, U$9.13, U$9.14, U$9.17, U$9.19, U$9.20, U$9.4, U$9.5, U$9.6
- removed net N$42: S1.3, U$2.VCC, U$5.4, U$9.18, U$9.2, U$9.3
- new net N$20: M2.1, U$2.D8
- new net N$28: M3.1, U$2.D9
- new net N$37: S1.3, U$2.GND, U$9.1, U$9.10, U$9.11, U$9.12, U$9.13, U$9.14, U$9.17, U$9.19, U$9.20, U$9.4, U$9.5, U$9.6
- new net N$4: C1.2, C2.2, C3.2, C4.2, J1.GND, J1.GNDBREAK, M1.2, M2.2, M3.2, PAD2.1, R1.3, R2.3, S1.1, U$1.3, U$1.4, U$2.GND1, U$2.VCC, U$5.3, U$5.4, U$6.SW2, U$7.SW2, U$8.SW2, U$9.18, U$9.2, U$9.3
- net N$11: now also J2.1; no longer M1.1
- net N$16: now also M1.1; no longer M2.1
- net N$17: now also J3.1; no longer M3.1
- net N$30: now also R4.2, U$2.A2; no longer R6.2, U$2.D8
- net N$31: now also R6.2, U$2.A3; no longer R4.2, U$2.D9
- net N$32: now also M1.3, M2.3, M3.3, OK1.3
- net N$33: now also OK1.13
- net N$34: no longer OK1.13
Routing:
- net N$38: track 206.3 -> 0.00 mm
- net N$4: track 0.00 -> 189.8 mm
- net N$42: track 108.3 -> 0.00 mm
- net N$37: track 0.00 -> 78.0 mm
- net N$32: track 0.00 -> 41.2 mm
- net N$20: track 0.00 -> 26.0 mm
- net N$28: track 0.00 -> 23.2 mm
- net N$30: track 39.1 -> 21.6 mm
- net N$31: track 32.1 -> 22.6 mm
- net N$23: track 7.62 -> 0.00 mm
- net N$11: track 28.0 -> 20.4 mm
- net N$16: track 25.0 -> 30.6 mm
- net N$17: track 21.2 -> 26.3 mm
- net N$6: track 23.5 -> 27.9 mm
- net N$21: track 41.4 -> 45.3 mm
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
Commit message: Cleaned up schematic and board layout
Parts:
- added FRAME1: FRAME-LETTER, SparkFun-Aesthetics:CREATIVE_COMMONS
Connections:
- net N$11 renamed SERVO_1_FEEDBACK
- net N$12 renamed BUTTON_3
- net N$13 renamed BUTTON_1
- net N$14 renamed BUTTON_2
- net N$15 renamed MODE_SWITCH
- net N$16 renamed SERVO_1_CONTROL
- net N$17 renamed SERVO_2_FEEDBACK
- net N$18 renamed MOSI
- net N$19 renamed DISP_RES
- net N$20 renamed SERVO_2_CONTROL
- net N$21 renamed MISO
- net N$22 renamed CS
- net N$25 renamed SCLK
- net N$28 renamed SERVO_3_CONTROL
- net N$30 renamed SHUTTER
- net N$31 renamed FOCUS
- removed net N$32: M1.3, M2.3, M3.3, OK1.2, OK1.3
- removed net N$37: S1.3, U$2.GND, U$9.1, U$9.10, U$9.11, U$9.12, U$9.13, U$9.14, U$9.17, U$9.19, U$9.20, U$9.4, U$9.5, U$9.6
- removed net N$4 (its old number): C1.2, C2.2, C3.2, C4.2, J1.GND, J1.GNDBREAK, M1.2, M2.2, M3.2, PAD2.1, R1.3, R2.3, S1.1, U$1.3, U$1.4, U$2.GND1, U$2.VCC, U$5.3, U$5.4, U$6.SW2, U$7.SW2, U$8.SW2, U$9.18, U$9.2, U$9.3
- removed net N$5 (its old number): C1.1, C3.1, J1.PWR, L1.1, L2.1, PAD1.1
- new net 5V: S1.1, U$2.VCC, U$5.4, U$9.18, U$9.2, U$9.3
- new net 6V: M1.2, M2.2, M3.2, U$1.4
- new net GND: C1.2, C2.2, C3.2, C4.2, J1.GND, J1.GNDBREAK, M1.3, M2.3, M3.3, OK1.2, OK1.3, R1.3, R2.3, S1.3, U$1.3, U$2.GND, U$2.GND1, U$5.3, U$6.SW2, U$7.SW2, U$8.SW2, U$9.1, U$9.10, U$9.11, U$9.12, U$9.13, U$9.14, U$9.17, U$9.19, U$9.20, U$9.4, U$9.5, U$9.6
- new net P+: C1.1, C3.1, J1.PWR, L1.1, L2.1
Routing:
- net GND: track 0.00 -> 197.6 mm
- net N$4 (its old number): track 189.8 -> 0.00 mm
- net 5V: track 0.00 -> 100.1 mm, vias 0 -> 1
- net N$37: track 78.0 -> 0.00 mm
- net N$5 (its old number): track 52.2 -> 0.00 mm
- net P+: track 0.00 -> 46.9 mm
- net N$32: track 41.2 -> 0.00 mm
- net 6V: track 0.00 -> 33.4 mm
- net SCLK: track 44.7 -> 42.5 mm
- net SHUTTER: track 21.6 -> 23.6 mm
- net MODE_SWITCH: track 35.3 -> 33.8 mm
