File: hardware/main_smd.brd (EAGLE design)
At the start: 269.8 x 110.3 mm, 192 parts, among them IC0 STM32F313VCT6, IC1 S1315F8_RAW, IC2 TMC262-LA, IC3 TMC262-LA, IC4 TMC262-LA, IC5 TMC424, IC6 TMC429-PI24, IC8 LM317MBSTT3, J1 POWER_JACKPTH_BREAD, J10 Motor Coil A, J11 Motor Coil B, J12 Motor Coil A, J3 Motor Coil B, J4 Motor Coil A, J5 73100-0114, J9 Motor Coil B, P1 1-2295018-2, U1 TPD8S300RUKRRUK0020B_NV, U2 FT232RL-REEL, U3 CDCS502PWR, U4 LSM9DS1, U5 TPS54336ADRCR, U6 TPS54336ADRCR, U7 TPS54336ADRCR, X1 STEREOJACK, Y1 7B-16.000MAAJ-T

Commit message: Updated hardware directory and other misc updates
Parts:
- moved C55 0.50 mm to (44.6, 19.6)
- renumbered D4 to D1, D6 to D2, D7 to D3, U$1 to Q3, U$10 to Q14, U$11 to Q11, U$12 to Q12, U$13 to Q9, U$14 to Q10, U$15 to Q15, U$16 to Q16, U$17 to Q7, U$18 to Q8, U$19 to Q19, U$2 to Q4, U$20 to Q20, U$21 to Q17, U$22 to Q18, U$23 to Q21, U$24 to Q22, U$25 to Q23, U$26 to Q24, U$5 to Q1, U$6 to Q2, U$7 to Q5, U$8 to Q6, U$9 to Q13
Connections:
- removed net 5V_OUT: IC2.9, IC3.9, IC4.9
- removed net NPOR: IC0.37
- removed net USART1_CK: IC0.67
- removed net USART1_CTS: IC0.70
- removed net USART1_RTS: IC0.71
- removed net USART2_CK: IC0.88
- removed net USB_SLAVE_A_RX2_N: P1.A10
- removed net USB_SLAVE_A_RX2_P: P1.A11
- removed net USB_SLAVE_A_TX1_N: P1.A3
- removed net USB_SLAVE_A_TX1_P: P1.A2
- removed net USB_SLAVE_B_RX1_N: P1.B10
- removed net USB_SLAVE_B_RX1_P: P1.B11
- removed net USB_SLAVE_B_TX2_N: P1.B3
- removed net USB_SLAVE_B_TX2_P: P1.B2
- removed net USB_S_OSC_IN: U2.27
- removed net USB_S_OSC_OUT: U2.28
Routing:
- net GND: track 526.0 -> 526.4 mm, vias 403 -> 402
Other:
- board text added: "All rights reserved"
- board text added: "Copyright Mel McCalla"
- board text added: "JTAG"
- board text added: "Panobot"
- board text added: "Version 0.1"
